File: hardware/reminder-sequin.kicad_sch (KiCad schematic)
At the start: 47 parts, among them J1 USB_C_Receptacle_USB2.0_16P, SW1 User, SW2 RST, SW3 BOOTSEL, U1 RP2040, U3 FM24C64B, U4 W25Q32JVSS, Y1 12MHz

Commit message: layout
Parts:
- C1, C10, C11, C12, C13, C14, C19, C2, C6, C7, C8, C9: footprint Capacitor_SMD:C_0603_1608Metric -> Capacitor_SMD:C_0402_1005Metric; LCSC Part # C14663 -> C1525
- C15, C16: footprint Capacitor_SMD:C_0603_1608Metric -> Capacitor_SMD:C_0402_1005Metric; LCSC Part # C1644 -> C1548
- R11, R21, R4, R8: footprint Resistor_SMD:R_0603_1608Metric -> Resistor_SMD:R_0402_1005Metric; LCSC Part # C21190 -> C11702
- R12, R14, R15, R16, R17, R19, R20: footprint Resistor_SMD:R_0603_1608Metric -> Resistor_SMD:R_0402_1005Metric; LCSC Part # C23186 -> C25905
- R18, R2, R22: footprint Resistor_SMD:R_0603_1608Metric -> Resistor_SMD:R_0402_1005Metric; LCSC Part # C25804 -> C25744
Connections:
- net LED: now also U1.15 (GPIO12)
Changed lines of the file:
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@@
 		)
 	)
+	(label "LED"
+		(at 127 77.47 0)
+		(effects
+			(font
+				(size 1.27 1.27)
+			)
+			(justify left bottom)
+		)
+	)
 	(label "USB_D-"
 		(at 195.58 66.04 0)
@@
 			)
 		)
-		(property "Footprint" "Capacitor_SMD:C_0603_1608Metric"
+		(property "Footprint" "Capacitor_SMD:C_0402_1005Metric"
 			(at 27.94 94.2848 0)
 			(effects
@@
 			)
 		)
-		(property "LCSC Part #" "C1644 "
+		(property "LCSC Part #" "C1548"
 			(at 24.13 95.25 0)
 			(effects
@@
 			)
 		)
-		(property "Footprint" "Resistor_SMD:R_0603_1608Metric"
+		(property "Footprint" "Resistor_SMD:R_0402_1005Metric"
 			(at 265.938 73.66 90)
 			(effects
@@
 			)
 		)
-		(property "LCSC Part #" "C23186 "
+		(property "LCSC Part #" "C25905"
 			(at 264.16 73.66 0)
 			(effects
@@
 			)
 		)
-		(property "Footprint" "Resistor_SMD:R_0603_1608Metric"
+		(property "Footprint" "Resistor_SMD:R_0402_1005Metric"
 			(at 173.482 123.19 90)
 			(effects
@@
 			)
 		)
-		(property "LCSC Part #" " C25804"
+		(property "LCSC Part #" " C25744"
 			(at 175.26 123.19 0)
 			(effects
@@
 			)
 		)
-		(property "Footprint" "Capacitor_SMD:C_0603_1608Metric"
+		(property "Footprint" "Capacitor_SMD:C_0402_1005Metric"
 			(at 91.44 25.7048 0)
 			(effects
@@
 			)
 		)
-		(property "LCSC Part #" "C14663"
+		(property "LCSC Part #" " C1525"
 			(at 87.63 26.67 0)
 			(effects
@@
 			)
 		)
-		(property "Footprint" "Capacitor_SMD:C_0603_1608Metric"
+		(property "Footprint" "Capacitor_SMD:C_0402_1005Metric"
 			(at 183.1848 21.59 0)
 			(effects
@@
 			)
 		)
-		(property "LCSC Part #" "C14663"
+		(property "LCSC Part #" " C1525"
 			(at 184.15 25.4 0)
 			(effects
@@
 			)
 		)
-		(property "Footprint" "Capacitor_SMD:C_0603_1608Metric"
+		(property "Footprint" "Capacitor_SMD:C_0402_1005Metric"
 			(at 148.8948 21.59 0)
 			(effects
@@
 			)
 		)
-		(property "LCSC Part #" "C14663"
+		(property "LCSC Part #" " C1525"
 			(at 149.86 25.4 0)
 			(effects
@@
 			)
 		)
-		(property "Footprint" "Resistor_SMD:R_0603_1608Metric"
+		(property "Footprint" "Resistor_SMD:R_0402_1005Metric"
 			(at 43.18 133.858 90)
 			(effects
@@
 			)
 		)
-		(property "LCSC Part #" "C21190"
+		(property "LCSC Part #" "C11702"
 			(at 43.18 132.08 0)
 			(effects
@@
 			)
 		)
-		(property "Footprint" "Resistor_SMD:R_0603_1608Metric"
+		(property "Footprint" "Resistor_SMD:R_0402_1005Metric"
 			(at 271.018 73.66 90)
 			(effects
@@
 			)
 		)
-		(property "LCSC Part #" "C23186 "
+		(property "LCSC Part #" "C25905"
 			(at 269.24 73.66 0)
 			(effects
@@
 			)
 		)
-		(property "Footprint" "Capacitor_SMD:C_0603_1608Metric"
+		(property "Footprint" "Capacitor_SMD:C_0402_1005Metric"
 			(at 171.7548 21.59 0)
 			(effects
@@
 			)
 		)
-		(property "LCSC Part #" "C14663"
+		(property "LCSC Part #" " C1525"
 			(at 172.72 25.4 0)
 			(effects
@@
 			)
 		)
-		(property "Footprint" "Resistor_SMD:R_0603_1608Metric"
+		(property "Footprint" "Resistor_SMD:R_0402_1005Metric"
 			(at 55.372 125.73 90)
 			(effects
@@
 			)
 		)
-		(property "LCSC Part #" " C25804"
+		(property "LCSC Part #" " C25744"
 			(at 57.15 125.73 0)
 			(effects
@@
 			)
 		)
-		(property "Footprint" "Capacitor_SMD:C_0603_1608Metric"
+		(property "Footprint" "Capacitor_SMD:C_0402_1005Metric"
 			(at 116.5352 181.61 0)
 			(effects
@@
 			)
 		)
-		(property "LCSC Part #" "C14663"
+		(property "LCSC Part #" " C1525"
 			(at 115.57 177.8 0)
 			(effects
@@
 			)
 		)
-		(property "Footprint" "Capacitor_SMD:C_0603_1608Metric"
+		(property "Footprint" "Capacitor_SMD:C_0402_1005Metric"
 			(at 137.4648 21.59 0)
 			(effects
@@
 			)
 		)
-		(property "LCSC Part #" "C14663"
+		(property "LCSC Part #" " C1525"
 			(at 138.43 25.4 0)
 			(effects
@@
 			)
 		)
-		(property "Footprint" "Capacitor_SMD:C_0603_1608Metric"
+		(property "Footprint" "Capacitor_SMD:C_0402_1005Metric"
 			(at 126.0348 21.59 0)
 			(effects
@@
 			)
 		)
-		(property "LCSC Part #" "C14663"
+		(property "LCSC Part #" " C1525"
 			(at 127 25.4 0)
 			(effects
@@
 			)
 		)
-		(property "Footprint" "Capacitor_SMD:C_0603_1608Metric"
+		(property "Footprint" "Capacitor_SMD:C_0402_1005Metric"
 			(at 91.44 37.1348 0)
 			(effects
@@
 			)
 		)
-		(property "LCSC Part #" "C14663"
+		(property "LCSC Part #" " C1525"
 			(at 87.63 38.1 0)
 			(effects
@@
 			)
 		)
-		(property "Footprint" "Resistor_SMD:R_0603_1608Metric"
+		(property "Footprint" "Resistor_SMD:R_0402_1005Metric"
 			(at 54.61 110.998 90)
 			(effects
@@
 			)
 		)
-		(property "LCSC Part #" "C21190"
+		(property "LCSC Part #" "C11702"
 			(at 54.61 109.22 0)
 			(effects
@@
 			)
 		)
-		(property "Footprint" "Capacitor_SMD:C_0603_1608Metric"
+		(property "Footprint" "Capacitor_SMD:C_0402_1005Metric"
 			(at 160.3248 21.59 0)
 			(effects
@@
 			)
 		)
-		(property "LCSC Part #" "C14663"
+		(property "LCSC Part #" " C1525"
 			(at 161.29 25.4 0)
 			(effects
@@
 			)
 		)
-		(property "Footprint" "Resistor_SMD:R_0603_1608Metric"
+		(property "Footprint" "Resistor_SMD:R_0402_1005Metric"
 			(at 126.238 162.56 90)
 			(effects
@@
 			)
 		)
-		(property "LCSC Part #" "C21190"
+		(property "LCSC Part #" "C11702"
 			(at 124.46 162.56 0)
 			(effects
@@
 			)
 		)
-		(property "Footprint" "Resistor_SMD:R_0603_1608Metric"
+		(property "Footprint" "Resistor_SMD:R_0402_1005Metric"
 			(at 208.28 62.738 90)
 			(effects
@@
 			)
 		)
-		(property "LCSC Part #" "C23186 "
+		(property "LCSC Part #" "C25905"
 			(at 208.28 60.96 0)
 			(effects
@@
 			)
 		)
-		(property "Footprint" "Resistor_SMD:R_0603_1608Metric"
+		(property "Footprint" "Resistor_SMD:R_0402_1005Metric"
 			(at 236.728 95.25 90)
 			(effects
@@
 			)
 		)
-		(property "LCSC Part #" "C23186 "
+		(property "LCSC Part #" "C25905"
 			(at 234.95 95.25 0)
 			(effects
@@
 			)
 		)
-		(property "Footprint" "Resistor_SMD:R_0603_1608Metric"
+		(property "Footprint" "Resistor_SMD:R_0402_1005Metric"
 			(at 231.648 95.25 90)
 			(effects
@@
 			)
 		)
-		(property "LCSC Part #" "C23186 "
+		(property "LCSC Part #" "C25905"
 			(at 229.87 95.25 0)
 			(effects
@@
 			)
 		)
-		(property "Footprint" "Resistor_SMD:R_0603_1608Metric"
+		(property "Footprint" "Resistor_SMD:R_0402_1005Metric"
 			(at 226.568 95.25 90)
 			(effects
@@
 			)
 		)
-		(property "LCSC Part #" "C23186 "
+		(property "LCSC Part #" "C25905"
 			(at 224.79 95.25 0)
 			(effects
@@
 			)
 		)
-		(property "Footprint" "Resistor_SMD:R_0603_1608Metric"
+		(property "Footprint" "Resistor_SMD:R_0402_1005Metric"
 			(at 208.28 60.198 90)
 			(effects
@@
 			)
 		)
-		(property "LCSC Part #" "C23186 "
+		(property "LCSC Part #" "C25905"
 			(at 208.28 58.42 0)
 			(effects
@@
 			)
 		)
-		(property "Footprint" "Capacitor_SMD:C_0603_1608Metric"
+		(property "Footprint" "Capacitor_SMD:C_0402_1005Metric"
 			(at 38.1 54.9148 0)
 			(effects
@@
 			)
 		)
-		(property "LCSC Part #" "C14663"
+		(property "LCSC Part #" " C1525"
 			(at 34.29 55.88 0)
 			(effects
@@
 			)
 		)
-		(property "Footprint" "Capacitor_SMD:C_0603_1608Metric"
+		(property "Footprint" "Capacitor_SMD:C_0402_1005Metric"
 			(at 27.94 108.2548 0)
 			(effects
@@
 			)
 		)
-		(property "LCSC Part #" "C1644 "
+		(property "LCSC Part #" "C1548"
 			(at 24.13 109.22 0)
 			(effects
@@
 			)
 		)
-		(property "Footprint" "Resistor_SMD:R_0603_1608Metric"
+		(property "Footprint" "Resistor_SMD:R_0402_1005Metric"
 			(at 200.152 127 90)
 			(effects
@@
 			)
 		)
-		(property "LCSC Part #" "C21190"
+		(property "LCSC Part #" "C11702"
 			(at 201.93 127 0)
 			(effects
@@
 			)
 		)
-		(property "Footprint" "Capacitor_SMD:C_0603_1608Metric"
+		(property "Footprint" "Capacitor_SMD:C_0402_1005Metric"
 			(at 236.22 75.8952 0)
 			(effects
@@
 			)
 		)
-		(property "LCSC Part #" "C14663"
+		(property "LCSC Part #" " C1525"
 			(at 240.03 74.93 0)
 			(effects
@@
 			)
 		)
-		(property "Footprint" "Resistor_SMD:R_0603_1608Metric"
+		(property "Footprint" "Resistor_SMD:R_0402_1005Metric"
 			(at 273.812 83.82 90)
 			(effects
@@
 			)
 		)
-		(property "LCSC Part #" " C25804"
+		(property "LCSC Part #" " C25744"
 			(at 275.59 83.82 0)
 			(effects
@@
 			)
 		)
-		(property "Footprint" "Capacitor_SMD:C_0603_1608Metric"
+		(property "Footprint" "Capacitor_SMD:C_0402_1005Metric"
 			(at 194.6148 21.59 0)
 			(effects
@@
 			)
 		)
-		(property "LCSC Part #" "C14663"
+		(property "LCSC Part #" " C1525"
 			(at 195.58 25.4 0)
 			(effects
